File: adcboard/adcboard.kicad_pcb (KiCad board)
At the start: 2 copper layers, 217.8 x 80.1 mm, 150 parts, among them J101 NegRail, J102 Detector, J103 PosRail, J107 FFRst, J108 ~DebReset, J109 ~DebA0, J110 SigOut, J111 ~DebCS, J112 DebCE, J401 TrigLvl, J403 SigADC, J406 ~DebArmed, J408 DebConv, J411 ~DebTrig, J501 SigInv, J502 SigDiff, J503 Sig1, J504 SigF1, J505 SigF2, J506 SigF3, U101 74HC04, U105 74HC04, U108 74HC04, U110 7400, U112 7400, U116 ADC-AD1674, U201 74LS138, U301 74LS374, U302 7400, U402 LT1016, U403 74HC74, U406 DG418, U407 74HC244, U408 AD8032, U501 LM6172, U502 AD744, U503 LM6172, U504 AD826

Commit message: Rev. 3 of ADC board, full 12V rail for analog
Parts:
- removed BUS101: A2_BUS, Apple2_bus:BUS_A2
- removed BlueLight: LED_Small, LEDs:LED_D5.0mm
- removed C103, C104, C111, C113, C115, C116, C117, C121, C125, C201, C301, C302: 2.2µF, Capacitors_THT:C_Disc_D3.8mm_W2.6mm_P2.50mm
- removed C109, C415: 100pF, Capacitors_THT:C_Disc_D3.8mm_W2.6mm_P2.50mm
- removed C401, C403, C407, C411, C504, C509: 10µF, Capacitors_THT:CP_Radial_D5.0mm_P2.50mm
- removed C402, C404, C408, C412, C505, C510, C514, C515, C522: 10nF, Capacitors_THT:C_Disc_D3.8mm_W2.6mm_P2.50mm
- removed C405: 150pF, Capacitors_THT:C_Disc_D3.8mm_W2.6mm_P2.50mm
- removed C406: 470pF, Capacitors_THT:C_Disc_D3.8mm_W2.6mm_P2.50mm
- removed C410, C414: 10pF, Capacitors_THT:C_Disc_D3.8mm_W2.6mm_P2.50mm
- removed C501, C506, C516, C517, C518: 470pF, Capacitors_THT:C_Rect_L7.0mm_W3.5mm_P5.00mm
- removed C502, C507, C511, C513, C519, C521: 2.2µF, Capacitors_THT:CP_Radial_D5.0mm_P2.50mm
- removed C503, C508, C512, C520: 100nF, Capacitors_THT:C_Disc_D3.8mm_W2.6mm_P2.50mm
- removed D110: D_Small, Diodes_THT:D_A-405_P7.62mm_Horizontal
- removed D301, D302, D303, D304, D305, D306, D307, D308: LED, LEDs:LED_D5.0mm
- removed D403, D404, D405: D, Diodes_THT:D_A-405_P7.62mm_Horizontal
- removed F101, F104: HC:250mA, Fuse_Holders_and_Fuses:Fuse_TE5_Littlefuse-395Series
- removed F102, F103: HC:160mA, Fuse_Holders_and_Fuses:Fuse_TE5_Littlefuse-395Series
- removed J101: NegRail, Pin_Headers:Pin_Header_Straight_1x03_Pitch2.54mm
- removed J102: Detector, Connectors_TE-Connectivity:BNC_Socket_TYCO-AMP_LargePads
- removed J103: PosRail, Pin_Headers:Pin_Header_Straight_1x03_Pitch2.54mm
- removed J107: FFRst, Pin_Headers:Pin_Header_Straight_1x02_Pitch2.54mm
- removed J108: ~DebReset, Socket_Strips:Socket_Strip_Straight_1x01_Pitch2.54mm
- removed J109: ~DebA0, Socket_Strips:Socket_Strip_Straight_1x01_Pitch2.54mm
- removed J110: SigOut, Pin_Headers:Pin_Header_Straight_1x03_Pitch2.54mm
- removed J111: ~DebCS, Socket_Strips:Socket_Strip_Straight_1x01_Pitch2.54mm
- removed J112: DebCE, Socket_Strips:Socket_Strip_Straight_1x01_Pitch2.54mm
- removed J401: TrigLvl, Pin_Headers:Pin_Header_Straight_1x03_Pitch2.54mm
- removed J403: SigADC, Pin_Headers:Pin_Header_Straight_1x03_Pitch2.54mm
- removed J406: ~DebArmed, Socket_Strips:Socket_Strip_Straight_1x01_Pitch2.54mm
- removed J408: DebConv, Socket_Strips:Socket_Strip_Straight_1x01_Pitch2.54mm
- removed J411: ~DebTrig, Socket_Strips:Socket_Strip_Straight_1x01_Pitch2.54mm
- removed J501: SigInv, Pin_Headers:Pin_Header_Straight_1x03_Pitch2.54mm
- removed J502: SigDiff, Pin_Headers:Pin_Header_Straight_1x03_Pitch2.54mm
- removed J503: Sig1, Pin_Headers:Pin_Header_Straight_1x03_Pitch2.54mm
- removed J504: SigF1, Pin_Headers:Pin_Header_Straight_1x03_Pitch2.54mm
- removed J505: SigF2, Pin_Headers:Pin_Header_Straight_1x03_Pitch2.54mm
- removed J506: SigF3, Pin_Headers:Pin_Header_Straight_1x03_Pitch2.54mm
- removed R116, R404, R502: 10k, Resistors_THT:R_Axial_DIN0207_L6.3mm_D2.5mm_P10.16mm_Horizontal
- removed R117, R118, R410, R412: 100, Resistors_THT:R_Axial_DIN0207_L6.3mm_D2.5mm_P10.16mm_Horizontal
- removed R122: 0(J), Resistors_THT:R_Axial_DIN0207_L6.3mm_D2.5mm_P10.16mm_Horizontal
- removed R127, R130: 50, Resistors_THT:R_Axial_DIN0207_L6.3mm_D2.5mm_P10.16mm_Horizontal
- removed R129, R201, R202, R309, R402, R407, R509: 4k7, Resistors_THT:R_Axial_DIN0207_L6.3mm_D2.5mm_P10.16mm_Horizontal
- removed R203: 0 (J), Resistors_THT:R_Axial_DIN0207_L6.3mm_D2.5mm_P10.16mm_Horizontal
- removed R301, R302, R303, R304, R305, R306, R307, R308, R401: 330, Resistors_THT:R_Axial_DIN0207_L6.3mm_D2.5mm_P10.16mm_Horizontal
- removed R408, R414: 6k2, Resistors_THT:R_Axial_DIN0207_L6.3mm_D2.5mm_P10.16mm_Horizontal
- removed R409: 100k, Resistors_THT:R_Axial_DIN0207_L6.3mm_D2.5mm_P10.16mm_Horizontal
- removed R411: 220, Resistors_THT:R_Axial_DIN0207_L6.3mm_D2.5mm_P10.16mm_Horizontal
- removed R415: 1k, Resistors_THT:R_Axial_DIN0207_L6.3mm_D2.5mm_P10.16mm_Horizontal
- removed R501: 150k, Resistors_THT:R_Axial_DIN0207_L6.3mm_D2.5mm_P10.16mm_Horizontal
- removed R503: 47k, Resistors_THT:R_Axial_DIN0207_L6.3mm_D2.5mm_P10.16mm_Horizontal
- removed R504, R505, R506, R507: 6k8, Resistors_THT:R_Axial_DIN0207_L6.3mm_D2.5mm_P10.16mm_Horizontal
- removed R508, R510, R511: 20k, Resistors_THT:R_Axial_DIN0207_L6.3mm_D2.5mm_P10.16mm_Horizontal
- removed R512, R513, R514: 15k, Resistors_THT:R_Axial_DIN0207_L6.3mm_D2.5mm_P10.16mm_Horizontal
- removed RV401: 50k, Potentiometers:Potentiometer_Trimmer_Bourns_3006P
- removed RV501: 100k, Potentiometers:Potentiometer_Trimmer_Bourns_3006P
- removed U101, U105, U108: 74HC04, Housings_DIP:DIP-14_W7.62mm
- removed U110, U112, U302: 7400, Housings_DIP:DIP-14_W7.62mm
- removed U116: ADC-AD1674, Housings_DIP:DIP-28_W15.24mm
- removed U201: 74LS138, Housings_DIP:DIP-16_W7.62mm
- removed U301: 74LS374, Housings_DIP:DIP-20_W7.62mm
- removed U402: LT1016, Housings_DIP:DIP-8_W7.62mm
- removed U403: 74HC74, Housings_DIP:DIP-14_W7.62mm
- removed U406: DG418, Housings_DIP:DIP-8_W7.62mm
- removed U407: 74HC244, Housings_DIP:DIP-20_W7.62mm
- removed U408: AD8032, Housings_DIP:DIP-8_W7.62mm
- removed U501, U503: LM6172, Housings_DIP:DIP-8_W7.62mm
- removed U502: AD744, Housings_DIP:DIP-8_W7.62mm
- removed U504: AD826, Housings_DIP:DIP-8_W7.62mm
- added BUS1: A2_BUS, ibxlib:BUS_ADC, F.Cu at (221.0, 146.1)
- added C1: 3.3µF, ibxlib:FG14, F.Cu at (167.3, 120.5)
- added C10: 10pF, ibxlib:FG18, F.Cu at (181.7, 130.5)
- added C11: 2.2nF, ibxlib:FG18, F.Cu at (178.5, 88.3)
- added C12: 10µF, ibxlib:FG16, F.Cu at (207.5, 102.3)
- added C13: 100nF, ibxlib:FG18, F.Cu at (230.2, 102.9)
- added C14: 10nF, ibxlib:FG18, F.Cu at (204.3, 98.7)
- added C15: 330pF, ibxlib:FG18, F.Cu at (160.4, 90.8)
- added C16: 10µF, ibxlib:FG16, F.Cu at (200.6, 99.9)
- added C17: 10µF, ibxlib:FG16, F.Cu at (193.7, 102.3)
- added C18: 10nF, ibxlib:FG18, F.Cu at (196.9, 98.6)
- added C19: 100nF, ibxlib:FG18, F.Cu at (219.1, 102.7)
- added C2: 3.3µF, ibxlib:FG14, F.Cu at (158.0, 134.9)
- added C20: 100nF, ibxlib:FG18, F.Cu at (229.9, 116.2)
- added C21: 100nF, ibxlib:FG18, F.Cu at (220.1, 75.8)
- added C22: 100nF, ibxlib:FG18, F.Cu at (258.6, 75.8)
- added C23: 100nF, ibxlib:FG18, F.Cu at (239.4, 75.8)
- added C24: 100nF, ibxlib:FG18, F.Cu at (157.6, 76.7)
- added C25: 100nF, ibxlib:FG18, F.Cu at (200.8, 75.8)
- added C26: 470pF, ibxlib:FG28, F.Cu at (93.2, 132.3)
- added C27: 2.2µF, ibxlib:FG14, F.Cu at (112.5, 118.5)
- added C28: 2.2µF, ibxlib:FG14, F.Cu at (103.5, 133.2)
- added C29: 10nF, ibxlib:FG18, F.Cu at (115.0, 124.1)
- added C3: 10nF, ibxlib:FG18, F.Cu at (169.6, 125.9)
- added C30: 10nF, ibxlib:FG18, F.Cu at (101.0, 127.7)
- added C31: 1µF, ibxlib:FG18, F.Cu at (118.3, 93.4)
- added C32: 1µF, ibxlib:FG18, F.Cu at (106.8, 107.7)
- added C33: 47pF, ibxlib:FG28, F.Cu at (104.8, 92.8)
- added C34: 100nF, ibxlib:FG18, F.Cu at (118.2, 98.8)
- added C35: 100nF, ibxlib:FG18, F.Cu at (104.3, 102.3)
- added C36: 470pF, ibxlib:FG28, F.Cu at (104.0, 116.7)
- added C37: 470pF, ibxlib:FG28, F.Cu at (122.4, 98.1)
- added C38: 2.2µF, ibxlib:FG14, F.Cu at (138.9, 86.0)
- added C39: 2.2µF, ibxlib:FG14, F.Cu at (129.1, 100.5)
- added C4: 10nF, ibxlib:FG18, F.Cu at (155.6, 129.5)
- added C40: 10nF, ibxlib:FG18, F.Cu at (141.1, 91.5)
- added C41: 10nF, ibxlib:FG18, F.Cu at (126.9, 95.0)
- added C42: 470pF, ibxlib:FG28, F.Cu at (132.2, 131.7)
- added C43: 3.3µF, ibxlib:FG14, F.Cu at (148.9, 116.7)
- added C44: 3.3µF, ibxlib:FG14, F.Cu at (139.9, 131.5)
- added C45: 10nF, ibxlib:FG18, F.Cu at (151.6, 122.2)
- added C46: 10nF, ibxlib:FG18, F.Cu at (137.3, 125.8)
- added C5: 100nF, ibxlib:FG18, F.Cu at (152.0, 104.6)
- added C6: 100nF, ibxlib:FG18, F.Cu at (151.9, 108.2)
- added C7: 10pF, ibxlib:FG18, F.Cu at (161.3, 120.6)
- added C8: 470pF, ibxlib:FG18, F.Cu at (182.1, 112.6)
- added C9: 100nF, ibxlib:FG18, F.Cu at (161.0, 99.3)
- added D1: SD103A, Diode_THT:D_DO-35_SOD27_P7.62mm_Horizontal, F.Cu at (167.9, 117.0)
- added D2: SD103A, Diode_THT:D_DO-35_SOD27_P7.62mm_Horizontal, F.Cu at (178.5, 116.9)
- added D3: SD103A, Diode_THT:D_DO-35_SOD27_P7.62mm_Horizontal, F.Cu at (179.3, 127.6)
- added D4: Blue Light, LED_THT:LED_D5.0mm, F.Cu at (185.7, 77.8)
- added D5: D_Zener_Small, Diode_THT:D_DO-35_SOD27_P7.62mm_Horizontal, F.Cu at (185.0, 117.6)
- added F1: HC:250mA, Fuse:Fuse_Littelfuse_395Series, F.Cu at (259.1, 130.8)
- added F2: HC:120mA, Fuse:Fuse_Littelfuse_395Series, F.Cu at (251.8, 135.9)
- added F3: HC:250mA, Fuse:Fuse_Littelfuse_395Series, F.Cu at (244.6, 135.9)
- added Gain: 100k, Potentiometer_THT:Potentiometer_Bourns_3006P_Horizontal, F.Cu at (144.7, 90.2)
- added J1: SigOut, ibxlib:3-Pin-Header, F.Cu at (152.1, 131.7)
- added J10: SigInv, ibxlib:3-Pin-Header, F.Cu at (141.2, 101.4)
- added J2: Detector, ibxlib:BNC_Socket_TYCO-AMP_LargePads, F.Cu at (94.1, 99.3)
- added J3: TrigLvl, ibxlib:3-Pin-Header, F.Cu at (148.5, 110.4)
- added J4: SigADC, ibxlib:3-Pin-Header, F.Cu at (185.5, 130.5)
- added J5: SigF1, ibxlib:3-Pin-Header, F.Cu at (100.1, 121.6)
- added J6: SigP, ibxlib:3-Pin-Header, F.Cu at (118.5, 107.0)
- added J7: SigF2, ibxlib:3-Pin-Header, F.Cu at (123.7, 124.1)
- added J8: SigDiff, ibxlib:3-Pin-Header, F.Cu at (130.1, 85.8)
- added J9: SigF3, ibxlib:3-Pin-Header, F.Cu at (143.8, 116.6)
- added R1: 6k8, ibxlib:Resistor, F.Cu at (155.6, 126.8)
- added R10: 10k, ibxlib:Resistor, F.Cu at (184.7, 94.7)
- added R11: 100, ibxlib:Resistor, F.Cu at (180.0, 97.9)
- added R12: 4k7, ibxlib:Resistor, F.Cu at (173.4, 91.3)
- added R13: 10k, ibxlib:Resistor, F.Cu at (163.2, 88.0)
- added R14: 4k7, ibxlib:Resistor, F.Cu at (259.7, 102.1)
- added R15: 4k7, ibxlib:Resistor, F.Cu at (256.4, 102.1)
- added R16: 4k7, ibxlib:Resistor, F.Cu at (259.7, 115.5)
- added R17: 4k7, ibxlib:Resistor, F.Cu at (213.6, 99.3)
- added R18: 49.9, ibxlib:Resistor, F.Cu at (180.0, 101.0)
- added R19: 49.9, ibxlib:Resistor, F.Cu at (190.8, 84.5)
- added R2: 47k, ibxlib:Resistor, F.Cu at (150.4, 96.1)
- added R20: 8k2, ibxlib:Resistor, F.Cu at (93.2, 122.8)
- added R21: 150k, ibxlib:Resistor, F.Cu at (112.2, 89.6)
- added R22: 20k, ibxlib:Resistor, F.Cu at (96.4, 122.8)
- added R23: 15k, ibxlib:Resistor, F.Cu at (96.4, 136.0)
- added R24: 8k2, ibxlib:Resistor, F.Cu at (110.3, 113.3)
- added R25: 8k2, ibxlib:Resistor, F.Cu at (122.4, 85.1)
- added R26: 20k, ibxlib:Resistor, F.Cu at (125.1, 128.9)
- added R27: 15k, ibxlib:Resistor, F.Cu at (115.0, 132.2)
- added R28: 10k, ibxlib:Resistor, F.Cu at (126.3, 81.4)
- added R29: 8k2, ibxlib:Resistor, F.Cu at (137.9, 122.7)
- added R3: 1k, ibxlib:Resistor, F.Cu at (173.1, 120.0)
- added R30: 47k, ibxlib:Resistor, F.Cu at (133.8, 75.6)
- added R31: 20k, ibxlib:Resistor, F.Cu at (127.7, 116.3)
- added R32: 15k, ibxlib:Resistor, F.Cu at (127.7, 119.5)
- added R33: 4k7, ibxlib:Resistor, F.Cu at (152.3, 135.3)
- added R4: 510, ibxlib:Resistor, F.Cu at (166.1, 110.2)
- added R5: 6k8, ibxlib:Resistor, F.Cu at (176.3, 130.1)
- added R6: 200, ibxlib:Resistor, F.Cu at (182.1, 127.5)
- added R7: 100, ibxlib:Resistor, F.Cu at (157.2, 82.0)
- added R8: 330, ibxlib:Resistor, F.Cu at (187.7, 84.5)
- added R9: 100, ibxlib:Resistor, F.Cu at (181.6, 94.7)
- added TP1: ~DebTrig, ibxlib:TP, F.Cu at (168.6, 73.7)
- added TP10: DebGND, ibxlib:TP, F.Cu at (191.3, 130.5)
- added TP11: ADC_STS, ibxlib:TP, F.Cu at (229.4, 129.1)
- added TP2: ~DebArmed, ibxlib:TP, F.Cu at (179.9, 73.7)
- added TP3: ~DebReset, ibxlib:TP, F.Cu at (253.1, 75.4)
- added TP4: ADC_VRef, ibxlib:TP, F.Cu at (175.3, 95.0)
- added TP5: DebConv, ibxlib:TP, F.Cu at (169.4, 94.9)
- added TP6: DebA0, ibxlib:TP, F.Cu at (206.6, 75.1)
- added TP7: DebCE, ibxlib:TP, F.Cu at (193.3, 75.1)
- added TP8: ~DebCS, ibxlib:TP, F.Cu at (197.8, 75.1)
- added TP9: DebGND, ibxlib:TP, F.Cu at (116.8, 83.2)
- added Trigger: 50k, Potentiometer_THT:Potentiometer_Bourns_3006P_Horizontal, F.Cu at (150.3, 90.2)
- added U1: AD826, ibxlib:DIP-8, F.Cu at (158.8, 123.9)
- added U10: ADC-AD1674, Package_DIP:DIP-28_W15.24mm_Socket, F.Cu at (221.0, 106.0)
- added U11: 74HCT244, Package_DIP:DIP-20_W7.62mm_Socket, F.Cu at (233.2, 124.3)
- added U12: LM6172, ibxlib:DIP-8, F.Cu at (104.1, 122.0)
- added U13: AD744, ibxlib:DIP-8, F.Cu at (107.5, 96.7)
- added U14: LM6172, ibxlib:DIP-8, F.Cu at (130.0, 89.4)
- added U15: AD826, ibxlib:DIP-8, F.Cu at (140.6, 120.2)
- added U2: DG418, ibxlib:DIP-8, F.Cu at (169.2, 102.7)
- added U3: AD790, ibxlib:DIP-8, F.Cu at (155.4, 102.6)
- added U4: 74HCT74, ibxlib:DIP-14, F.Cu at (161.0, 84.8)
- added U5: 74HCT04, ibxlib:DIP-14, F.Cu at (195.2, 79.2)
- added U6: 74HCT00, ibxlib:DIP-14, F.Cu at (253.0, 79.2)
- added U7: 74HCT00, ibxlib:DIP-14, F.Cu at (214.5, 79.2)
- added U8: 74HCT138, Package_DIP:DIP-16_W7.62mm_Socket, F.Cu at (233.3, 110.9)
- added U9: 74HCT04, ibxlib:DIP-14, F.Cu at (233.8, 79.2)
Routing:
- net Net-(J107-Pad1): track 135.2 -> 0.00 mm, vias 3 -> 0
- net -5V: track 134.1 -> 0.00 mm
- net +Rail: track 115.7 -> 0.00 mm, vias 2 -> 0
- net Net-(TP3-Pad1): track 0.00 -> 108.9 mm, vias 0 -> 2
- net -12V: track 314.3 -> 419.4 mm, vias 1 -> 4
- net Net-(D110-Pad2): track 102.8 -> 0.00 mm, vias 2 -> 0
- net Net-(U301-Pad11): track 87.1 -> 0.00 mm, vias 1 -> 0
- net -Rail: track 81.5 -> 0.00 mm
- net Net-(R12-Pad1): track 0.00 -> 80.4 mm, vias 0 -> 2
- net WR: track 78.4 -> 0.00 mm, vias 1 -> 0
- net Net-(U5-Pad9): track 0.00 -> 74.9 mm, vias 0 -> 6
- net ~BufferOE: track 136.6 -> 63.6 mm, vias 3 -> 2
- net D7: track 160.2 -> 87.9 mm, vias 4 -> 3
- net Net-(D301-Pad2): track 66.7 -> 0.00 mm
- net Net-(D308-Pad2): track 66.3 -> 0.00 mm
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Other:
- board size 217.8 x 80.1 mm -> 184 x 80 mm
- net class Default: trace_width 0.25 -> 0.254; via_dia 0.6 -> 0.635; via_drill 0.4 -> 0.381
- net class Power: trace_width 0.4 -> 0.381; via_dia 0.6 -> 0.635; via_drill 0.4 -> 0.381
- board text added: "IBX II ADC Board (Rev. 3 "Supermicro")"
- board text added: "Moritz Kütt Princeton University"
- board text removed: "+12V"
- board text removed: "+5V"
- board text removed: "-12V"
- board text removed: "-5V"
- board text removed: "IBX ][ 12 Bit (Rev.1) Made up in J207"
