File: hvboard/hvboard.kicad_pcb (KiCad board)
At the start: 2 copper layers, 145 x 80 mm, 51 parts, among them J101 Debug-1, J102 HV, J103 Debug-2, U101 AD584, U102 74LS14, U103 74HC74, U104 7400, U105 7400, U106 74LS374, U107 CHV, U108 74LS138

Commit message: HV board - KiCad 5 and small footprint changes
Parts:
- C101, C103, C105, C106, C107, C109, C110: footprint Capacitors_THT:C_Rect_L4.0mm_W2.5mm_P2.50mm -> ibxlib:FG18
- C104, C108: footprint Capacitors_THT:C_Rect_L4.0mm_W2.5mm_P2.50mm -> ibxlib:FG14
- R101, R102, R104, R106, R108, R110, R112, R114, R116, R117, R118, R119, R120, R121, R122, R123, R124, R128: footprint Resistors_THT:R_Axial_DIN0207_L6.3mm_D2.5mm_P10.16mm_Horizontal -> ibxlib:Resistor
- R103, R105, R107, R109, R111, R113, R115: value 10k -> 10k+; footprint Resistors_THT:R_Axial_DIN0207_L6.3mm_D2.5mm_P10.16mm_Horizontal -> ibxlib:Resistor
- R125: value 0 -> 4k7; footprint Resistors_THT:R_Axial_DIN0207_L6.3mm_D2.5mm_P10.16mm_Horizontal -> ibxlib:Resistor
- U101: footprint Housings_DIP:DIP-8_W7.62mm -> ibxlib:DIP-8
- U102: value 74LS14 -> 74HCT14; footprint Housings_DIP:DIP-14_W7.62mm -> ibxlib:DIP-14
- U103: value 74HC74 -> 74HCT74; footprint Housings_DIP:DIP-14_W7.62mm -> ibxlib:DIP-14
- U104, U105: value 7400 -> 74HCT00; footprint Housings_DIP:DIP-14_W7.62mm -> ibxlib:DIP-14
- U108: value 74LS138 -> 74HCT138
- moved R119 10.3 mm to (155.2, 74.7), turned to 180 degrees
- moved C107 2.59 mm to (187.3, 81.6), turned to 90 degrees
- moved C101 2.58 mm to (169.2, 91.3), turned to 90 degrees
- moved C104 2.56 mm to (160.5, 82.5), turned to 180 degrees
- moved C106 2.56 mm to (187.4, 94.5), turned to 90 degrees
- moved C103 2.52 mm to (187.3, 68.7), turned to 90 degrees
- moved C105 2.27 mm to (159.7, 72.7), turned to 90 degrees
- moved C108 1.71 mm to (141.8, 88.3), turned to 270 degrees
Connections:
- C103 pad 1: +5V -> GND
- C103 pad 2: GND -> +5V
- C104 pad 1: Net-(C104-Pad1) -> GND
- C104 pad 2: GND -> Net-(C104-Pad2)
- C105 pad 1: +5V -> GND
- C105 pad 2: GND -> +5V
- C106 pad 1: +5V -> GND
- C106 pad 2: GND -> +5V
- C107 pad 1: +5V -> GND
- C107 pad 2: GND -> +5V
- C108 pad 1: Net-(C108-Pad1) -> GND
- C108 pad 2: GND -> Net-(C108-Pad2)
- J103 pad 1: Net-(C108-Pad1) -> Net-(C108-Pad2)
- R119 pad 1: Net-(D101-Pad1) -> GND
- R119 pad 2: GND -> Net-(D101-Pad1)
- R122 pad 2: Net-(C108-Pad1) -> Net-(C108-Pad2)
- R124 pad 1: Net-(C108-Pad1) -> Net-(C108-Pad2)
- U101 pad 1: Net-(C104-Pad1) -> Net-(C104-Pad2)
- U101 pad 2: Net-(C104-Pad1) -> Net-(C104-Pad2)
- U101 pad 6: Net-(C101-Pad2) -> Net-(C101-Pad1)
- U101 pad 7: Net-(C101-Pad1) -> Net-(C101-Pad2)
- U106 pad 20: Net-(C104-Pad1) -> Net-(C104-Pad2)
- U107 pad 4: Net-(C108-Pad1) -> Net-(C108-Pad2)
Routing:
- net Net-(C108-Pad1): track 56.4 -> 0.00 mm
- net Net-(C108-Pad2): track 0.00 -> 54.4 mm
- net Net-(C104-Pad1): track 19.2 -> 0.00 mm
- net Net-(C104-Pad2): track 0.00 -> 19.0 mm
